File: shield/Shield/Shield.kicad_sch (KiCad schematic)
At the start: 33 parts, among them J1 Conn_02x20_Counter_Clockwise, J2 Conn_02x20_Counter_Clockwise, J3 DE15_Receptacle_HighDensity, SW1 SW_Push, SW2 SW_Push, SW3 SW_Push, SW4 SW_Push, SW5 SW_DPST_x2, SW6 SW_DPST_x2, SW7 SW_DPST_x2, SW8 SW_DPST_x2, U1 HDSP-7401, U2 HDSP-7401, U3 HDSP-7401, U4 HDSP-7401, U5 HDSP-7401, U6 HDSP-7401

Commit message: Avance en la PCB
Parts:
- removed J3: DE15_Receptacle_HighDensity, symbol Connector:DE15_Receptacle_HighDensity
- added C1, C10, C11, C12, C2, C3, C9: C, symbol Device:C
- added C4: 10u, symbol Device:C
- added J3: Jack-DC, symbol Connector:Jack-DC
- added J4: Conn_01x08, symbol Connector_Generic:Conn_01x08
- added J5: DE15_Receptacle_HighDensity_MountingHoles, symbol Connector:DE15_Receptacle_HighDensity_MountingHoles
- added R10, R11, R12, R13, R14, R15, R16, R17, R18, R19, R20, R21, R22, R23, R24, R25, R26, R27, R9: R, symbol Device:R
- added RN1, RN10, RN12, RN3, RN4, RN8: 100, symbol Device:R_Pack04
- added RN11, RN13, RN2, RN5, RN6, RN9: R_Pack04, symbol Device:R_Pack04
- added U7: ADV7123JSTZ240-RL, ST_48_ADI, symbol ADC:ADV7123JSTZ240-RL
- added U8: OKI-78SR-3.3_1.5-W36-C, Converter_DCDC:Converter_DCDC_Murata_OKI-78SR_Vertical, symbol Converter_DCDC:OKI-78SR-3.3_1.5-W36-C
Connections:
- net VSS: now reaches U4.1 (CA)
- net VSS: now also R1.1, R2.1, R3.1, R4.1, R5.1, R6.1, R7.1, R8.1, U1.1 (CA), U1.6 (CA), U2.1 (CA), U2.6 (CA), U3.1 (CA), U3.6 (CA), U4.6 (CA), U5.1 (CA), U5.6 (CA), U6.1 (CA), U6.6 (CA), C10.1, C11.1, C12.1, C2.1, C3.1, C4.1, C9.1, R10.1, R11.1, R12.1, R13.1, R14.1, R15.1, R16.1, R17.1, R18.1, R19.1, R20.1, R26.2, R9.1, U7.13 (VAA), U7.29 (VAA), U7.30 (VAA), U8.3 (OUT)
- net at U4.10 (A): now also RN8.4 (R4.1)
- net at U4.2 (F): now also RN9.3 (R3.1)
- net at U4.3 (G): now also RN9.2 (R2.1)
- net at U4.4 (E): now also RN9.4 (R4.1)
- net at U4.5 (D): now also RN8.1 (R1.1)
- net at U4.7 (DP): now also RN9.1 (R1.1)
- net at U4.8 (C): now also RN8.2 (R2.1)
- net at U4.9 (B): now also RN8.3 (R3.1)
- net GND: now reaches SW4.1
- net GND: now also SW1.1, SW2.1, SW3.1, SW5.1 (A), SW5.3 (A), SW6.1 (A), SW6.3 (A), SW7.1 (A), SW7.3 (A), SW8.1 (A), SW8.3 (A), C1.2, C4.2, J3.2, J5.10, J5.5, J5.6, J5.7, J5.8, R21.1, R22.2, R23.2, R27.2, U7.1 (G0), U7.14 (B0), U7.15 (B1), U7.2 (G1), U7.25 (GND), U7.26 (GND), U7.27 (IOB*), U7.31 (IOG*), U7.33 (IOR*), U7.39 (R0), U7.40 (R1), U8.2 (GND)
- net P_3: now reaches SW4.2
- net P_3: now also C12.2, R20.2
- net LED_2: now reaches D3.1 (K)
- net at D3.2 (A): now also R3.2
- net SW_0: now reaches SW8.4 (B)
- net SW_0: now also SW5.2 (B), SW5.4 (B), SW6.2 (B), SW6.4 (B), SW7.2 (B), SW7.4 (B), SW8.2 (B), R10.2, R11.2, R12.2, R13.2, R14.2, R15.2, R16.2, R9.2
- net LED_4: now reaches D5.1 (K)
- net at D5.2 (A): now also R5.2
- net LED_3: now reaches D4.1 (K)
- net at D4.2 (A): now also R4.2
- net at U1.10 (A): now also RN1.4 (R4.1)
- net at U1.2 (F): now also RN2.3 (R3.1)
- net at U1.3 (G): now also RN2.2 (R2.1)
- net at U1.4 (E): now also RN2.4 (R4.1)
- net at U1.5 (D): now also RN1.1 (R1.1)
- net at U1.7 (DP): now also RN2.1 (R1.1)
- net at U1.8 (C): now also RN1.2 (R2.1)
- net at U1.9 (B): now also RN1.3 (R3.1)
- net P_2: now reaches SW3.2
- net P_2: now also C11.2, R19.2
- net at U3.10 (A): now also RN3.4 (R4.1)
- net at U3.2 (F): now also RN6.3 (R3.1)
- net at U3.3 (G): now also RN6.2 (R2.1)
- net at U3.4 (E): now also RN6.4 (R4.1)
- net at U3.5 (D): now also RN3.1 (R1.1)
- net at U3.7 (DP): now also RN6.1 (R1.1)
- net at U3.8 (C): now also RN3.2 (R2.1)
- net at U3.9 (B): now also RN3.3 (R3.1)
- net at R8.2: now also D8.2 (A)
- net at U6.10 (A): now also RN12.4 (R4.1)
- net at U6.2 (F): now also RN13.3 (R3.1)
- net at U6.3 (G): now also RN13.2 (R2.1)
- net at U6.4 (E): now also RN13.4 (R4.1)
- net at U6.5 (D): now also RN12.1 (R1.1)
- net at U6.7 (DP): now also RN13.1 (R1.1)
- net at U6.8 (C): now also RN12.2 (R2.1)
- net at U6.9 (B): now also RN12.3 (R3.1)
- net at U2.10 (A): now also RN4.4 (R4.1)
- net at U2.2 (F): now also RN5.3 (R3.1)
- net at U2.3 (G): now also RN5.2 (R2.1)
- net at U2.4 (E): now also RN5.4 (R4.1)
- net at U2.5 (D): now also RN4.1 (R1.1)
- net at U2.7 (DP): now also RN5.1 (R1.1)
- net at U2.8 (C): now also RN4.2 (R2.1)
- net at U2.9 (B): now also RN4.3 (R3.1)
- net at R2.2: now also D2.2 (A)
- net at R7.2: now also D7.2 (A)
- net LED_1: now reaches D2.1 (K)
- net at U5.10 (A): now also RN10.4 (R4.1)
- net at U5.2 (F): now also RN11.3 (R3.1)
- net at U5.3 (G): now also RN11.2 (R2.1)
- net at U5.4 (E): now also RN11.4 (R4.1)
- net at U5.5 (D): now also RN10.1 (R1.1)
- net at U5.7 (DP): now also RN11.1 (R1.1)
- net at U5.8 (C): now also RN10.2 (R2.1)
- net at U5.9 (B): now also RN10.3 (R3.1)
- net LED_5: now reaches D6.1 (K)
- net at D6.2 (A): now also R6.2
- net P_0: now reaches SW1.2
- net P_0: now also C9.2, R17.2
- net LED_0: now reaches D1.1 (K)
- net at D1.2 (A): now also R1.2
- net LED_7: now reaches D8.1 (K)
- net LED_6: now reaches D7.1 (K)
- net P_1: now reaches SW2.2
- net P_1: now also C10.2, R18.2
- new net: C1.1, J5.0
- new net: J5.13, R24.1
- new net: J5.1, R21.2, U7.34 (IOR)
- new net: J5.14, R25.1
- new net: J5.2, R22.1, U7.32 (IOG)
- new net: J5.3, R23.1, U7.28 (IOB)
- new net: J3.1, U8.1 (IN)
- new net: C2.2, U7.35 (COMP)
- new net: R26.1, U7.38 (PSAVE*)
- new net: C3.2, U7.36 (VREF)
- new net: R27.1, U7.37 (RSET)
- new net HEX_00: RN1.5 (R4.2)
- new net HEX_01: RN1.6 (R3.2)
- new net HEX_02: RN1.7 (R2.2)
- new net HEX_03: RN1.8 (R1.2)
- new net HEX_04: RN2.5 (R4.2)
- new net HEX_05: RN2.6 (R3.2)
- new net HEX_06: RN2.7 (R2.2)
- new net HEX_07: RN2.8 (R1.2)
- new net HEX_10: RN4.5 (R4.2)
- new net HEX_11: RN4.6 (R3.2)
- new net HEX_12: RN4.7 (R2.2)
- new net HEX_13: RN4.8 (R1.2)
- new net HEX_14: RN5.5 (R4.2)
- new net HEX_15: RN5.6 (R3.2)
- new net HEX_16: RN5.7 (R2.2)
- new net HEX_17: RN5.8 (R1.2)
- new net HEX_20: RN3.5 (R4.2)
- new net HEX_21: RN3.6 (R3.2)
- new net HEX_22: RN3.7 (R2.2)
- new net HEX_23: RN3.8 (R1.2)
- new net HEX_24: RN6.5 (R4.2)
- new net HEX_25: RN6.6 (R3.2)
- new net HEX_26: RN6.7 (R2.2)
- new net HEX_27: RN6.8 (R1.2)
- new net HEX_30: RN8.5 (R4.2)
- new net HEX_31: RN8.6 (R3.2)
- new net HEX_32: RN8.7 (R2.2)
- new net HEX_33: RN8.8 (R1.2)
- new net HEX_34: RN9.5 (R4.2)
- new net HEX_35: RN9.6 (R3.2)
- new net HEX_36: RN9.7 (R2.2)
- new net HEX_37: RN9.8 (R1.2)
- new net HEX_40: RN10.5 (R4.2)
- new net HEX_41: RN10.6 (R3.2)
- new net HEX_42: RN10.7 (R2.2)
- new net HEX_43: RN10.8 (R1.2)
- new net HEX_44: RN11.5 (R4.2)
- new net HEX_45: RN11.6 (R3.2)
- new net HEX_46: RN11.7 (R2.2)
- new net HEX_47: RN11.8 (R1.2)
- new net HEX_50: RN12.5 (R4.2)
- new net HEX_51: RN12.6 (R3.2)
- new net HEX_52: RN12.7 (R2.2)
- new net HEX_53: RN12.8 (R1.2)
- new net HEX_54: RN13.5 (R4.2)
- new net HEX_55: RN13.6 (R3.2)
- new net HEX_56: RN13.7 (R2.2)
- new net HEX_57: RN13.8 (R1.2)
- new net T_0: J4.1 (Pin_1)
- new net T_1: J4.2 (Pin_2)
- new net T_2: J4.3 (Pin_3)
- new net T_3: J4.4 (Pin_4)
- new net T_4: J4.5 (Pin_5)
- new net T_5: J4.6 (Pin_6)
- new net T_6: J4.7 (Pin_7)
- new net T_7: J4.8 (Pin_8)
- new net VGA_B0: U7.16 (B2)
- new net VGA_B1: U7.17 (B3)
- new net VGA_B2: U7.18 (B4)
- new net VGA_B3: U7.19 (B5)
- new net VGA_B4: U7.20 (B6)
- new net VGA_B5: U7.21 (B7)
- new net VGA_B6: U7.22 (B8)
- new net VGA_B7: U7.23 (B9)
- new net VGA_BLANK: U7.11 (BLANK*)
- new net VGA_CLK: U7.24 (CLOCK)
- new net VGA_G0: U7.3 (G2), U7.41 (R2)
- new net VGA_G1: U7.4 (G3), U7.42 (R3)
- new net VGA_G2: U7.43 (R4), U7.5 (G4)
- new net VGA_G3: U7.44 (R5), U7.6 (G5)
- new net VGA_G4: U7.45 (R6), U7.7 (G6)
- new net VGA_G5: U7.46 (R7), U7.8 (G7)
- new net VGA_G6: U7.47 (R8), U7.9 (G8)
- new net VGA_G7: U7.10 (G9), U7.48 (R9)
- new net VGA_HS: R24.2
- new net VGA_SYNC: U7.12 (SYNC*)
- new net VGA_VS: R25.2
Other:
- note added: "Teclado"
- note added: "total pines 68+VGA+TECLADO"
- moved on the sheet: D1, D2, D3, D4, D5, D6, D7, D8, J1, J2, R1, R2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
